Commit message: add gazebo properties

File: src/elephant/elerobot_description/xacro/color.xacro (robot description, xacro)
@@ -7,7 +7,12 @@
     </gazebo>
   </xacro:macro>
-  <xacro:macro name="gazebo_black" params="link">
+  <xacro:macro name="gazebo_grey" params="link">
     <gazebo reference="${link}">
-      <material>Gazebo/Black</material>
+      <material>Gazebo/Grey</material>
+    </gazebo>
+  </xacro:macro>
+  <xacro:macro name="gazebo_red" params="link">
+    <gazebo reference="${link}">
+      <material>Gazebo/Red</material>
       <mu1>0.61</mu1>
       <mu2>0.47</mu2>

File: src/elephant/elerobot_description/xacro/elerobot_unit.urdf.xacro (robot description, xacro)
@@ -10,4 +10,20 @@
   <xacro:if value="$(arg gazebo)">
     <xacro:elerobot arm_id="${arm_id}" with_camera="$(arg with_camera)"/>
+    <!-- gazebo color -->
+    <xacro:gazebo_white link="${arm_id}_link0"/>
+    <xacro:gazebo_white link="${arm_id}_link1"/>
+    <xacro:gazebo_white link="${arm_id}_link2"/>
+    <xacro:gazebo_white link="${arm_id}_link3"/>
+    <xacro:gazebo_white link="${arm_id}_link4"/>
+    <xacro:gazebo_white link="${arm_id}_link5"/>
+    <xacro:gazebo_grey  link="${arm_id}_link6"/>
+    <xacro:gazebo_red   link="${arm_id}_link6"/>
+    <!-- gazebo joint hardware interface -->
+    <xacro:gazebo-joint joint="${arm_id}_joint0" transmission="hardware_interface/PositionJointInterface" />
+    <xacro:gazebo-joint joint="${arm_id}_joint1" transmission="hardware_interface/PositionJointInterface" />
+    <xacro:gazebo-joint joint="${arm_id}_joint2" transmission="hardware_interface/PositionJointInterface" />
+    <xacro:gazebo-joint joint="${arm_id}_joint3" transmission="hardware_interface/PositionJointInterface" />
+    <xacro:gazebo-joint joint="${arm_id}_joint4" transmission="hardware_interface/PositionJointInterface" />
+    <xacro:gazebo-joint joint="${arm_id}_joint5" transmission="hardware_interface/PositionJointInterface" />
     <!-- Gazebo plugin for ROS control -->
     <gazebo>
