Commit message: upgrade the parameters accurancy of the model

File: src/elephant/elerobot_description/xacro/elerobot.xacro (robot description, xacro)
@@ -41,5 +41,5 @@
     <link name="${arm_id}_link1">
       <visual>
-        <origin xyz="-0.051 -0.051 -0.07" rpy="0.0 0.0 0.0"/>
+        <origin xyz="-0.0528 -0.0528 -0.07" rpy="0.0 0.0 0.0"/>
         <geometry>
           <mesh filename="${mesh_file_path}${mesh_prefix}1${mesh_suffix}" scale="0.001 0.001 0.001"/>
@@ -65,5 +65,5 @@
     <link name="${arm_id}_link2">
       <visual>
-        <origin xyz="-0.0525 -0.0525 0.154" rpy="${-PI/2} 0.0 0.0"/>
+        <origin xyz="-0.054 -0.053 0.154" rpy="${-PI/2} 0.0 0.0"/>
         <geometry>
           <mesh filename="${mesh_file_path}${mesh_prefix}2${mesh_suffix}" scale="0.001 0.001 0.001"/>
@@ -72,5 +72,5 @@
       </visual>
       <collision>
-        <origin xyz="-0.05 -0.05 0.154" rpy="${-PI/2} 0.0 0.0"/>
+        <origin xyz="-0.054 -0.053 0.154" rpy="${-PI/2} 0.0 0.0"/>
         <geometry>
           <mesh filename="${mesh_file_path}${mesh_prefix}2${mesh_suffix}" scale="0.001 0.001 0.001"/>
@@ -89,5 +89,5 @@
     <link name="${arm_id}_link3">
       <visual>
-        <origin xyz="0.284 0.078 0.025" rpy="${-PI/2} 0.0 ${PI}"/>
+        <origin xyz="0.2815 0.078 0.024" rpy="${-PI/2} 0.0 ${PI}"/>
         <geometry>
           <mesh filename="${mesh_file_path}${mesh_prefix}3${mesh_suffix}" scale="0.001 0.001 0.001"/>
@@ -96,5 +96,5 @@
       </visual>
       <collision>
-        <origin xyz="0.284 0.078 0.025" rpy="${-PI/2} 0.0 ${PI}"/>
+        <origin xyz="0.2815 0.078 0.024" rpy="${-PI/2} 0.0 ${PI}"/>
         <geometry>
           <mesh filename="${mesh_file_path}${mesh_prefix}3${mesh_suffix}" scale="0.001 0.001 0.001"/>
@@ -113,5 +113,5 @@
     <link name="${arm_id}_link4">
       <visual>
-        <origin xyz="-0.078 -0.06 0.045" rpy="${-PI/2} 0.0 0.0"/>
+        <origin xyz="-0.0772 -0.0596 0.044" rpy="${-PI/2} 0.0 0.0"/>
         <geometry>
           <mesh filename="${mesh_file_path}${mesh_prefix}4${mesh_suffix}" scale="0.001 0.001 0.001"/>
@@ -120,5 +120,5 @@
       </visual>
       <collision>
-        <origin xyz="-0.078 -0.06 0.045" rpy="${-PI/2} 0.0 0.0"/>
+        <origin xyz="-0.0772 -0.0596 0.044" rpy="${-PI/2} 0.0 0.0"/>
         <geometry>
           <mesh filename="${mesh_file_path}${mesh_prefix}4${mesh_suffix}" scale="0.001 0.001 0.001"/>
@@ -137,5 +137,5 @@
     <link name="${arm_id}_link5">
       <visual>
-        <origin xyz="0.078 0.061 0.046" rpy="${-PI/2} 0.0 ${PI}"/>
+        <origin xyz="0.0775 0.0605 0.046" rpy="${-PI/2} 0.0 ${PI}"/>
         <geometry>
           <mesh filename="${mesh_file_path}${mesh_prefix}5${mesh_suffix}" scale="0.001 0.001 0.001"/>
@@ -144,5 +144,5 @@
       </visual>
       <collision>
-        <origin xyz="0.078 0.061 0.046" rpy="${-PI/2} 0.0 ${PI}"/>
+        <origin xyz="0.0775 0.0605 0.046" rpy="${-PI/2} 0.0 ${PI}"/>
         <geometry>
           <mesh filename="${mesh_file_path}${mesh_prefix}5${mesh_suffix}" scale="0.001 0.001 0.001"/>
@@ -161,23 +161,43 @@
     <link name="${arm_id}_link6">
       <visual>
-        <origin xyz="0.0 0.0 0.0" rpy="0.0 0.0 0.0"/>
+        <origin xyz="-0.0425 -0.0425 -0.007" rpy="0.0 0.0 0.0"/>
         <geometry>
           <mesh filename="${mesh_file_path}${mesh_prefix}6${mesh_suffix}" scale="0.001 0.001 0.001"/>
         </geometry>
-        <material name="white"/>
-      </visual>
-      <collision>
-        <origin xyz="0.0 0.0 0.0" rpy="0.0 0.0 0.0"/>
+        <material name="grey"/>
+      </visual>
+      <collision>
+        <origin xyz="-0.0425 -0.0425 -0.007" rpy="0.0 0.0 0.0"/>
         <geometry>
           <mesh filename="${mesh_file_path}${mesh_prefix}6${mesh_suffix}" scale="0.001 0.001 0.001"/>
         </geometry>
-        <material name="white"/>
+        <material name="grey"/>
       </collision>
       <inertial>
         <origin xyz="-0.0001 -0.00033 0.02" rpy="0.0 0.0 0.0"/>
         <mass value="${link6_mass}"/>
-        <inertia ixx="0.0003" ixy="0.0" ixz="0.0000"
-                              iyy="0.0003" iyz="0.0002"
-                                         izz="0.0003"/>
+        <inertia ixx="0.0003" ixy="0.0"    ixz="0.0"
+                              iyy="0.0003" iyz="0.0"
+                                           izz="0.0003"/>
+      </inertial>
+    </link>
+    <link name="${arm_id}_link7">
+      <visual>
+        <origin xyz="0.0 0.0 ${-link7_h/2}" rpy="0.0 0.0 0.0"/>
+        <geometry>
+          <cylinder radius="${link7_r}" length="${link7_h}"/>
+        </geometry>
+        <material name="red"/>
+      </visual>
+      <collision>
+        <origin xyz="0.0 0.0 0.0" rpy="0.0 0.0 0.0"/>
+        <geometry>
+          <cylinder radius="${link7_r}" length="${link7_h}"/>
+        </geometry>
+      </collision>
+      <inertial>
+          <origin xyz="0.0 0.0 0.0" rpy="0.0 0.0 0.0"/>
+          <mass value="${link7_mass}"/>
+          <xacro:cylinder_inertia m="${link7_mass}" r="${link7_r}" h="${link7_h}"/>
       </inertial>
     </link>
@@ -233,4 +253,20 @@
       <dynamics D="1" K="7000" mu_coulomb="0" mu_viscous="16" damping="0.003" friction="0.01"/>
     </joint>
+    <!-- joint5 -->
+    <joint name="${arm_id}_joint5" type="revolute">
+      <axis xyz="0 0 1"/>
+      <origin xyz="0.0 ${joint5_y} 0.0" rpy="${-PI/2} 0.0 0.0"/>
+      <safety_controller k_position="50.0" k_velocity="20.0" soft_lower_limit="${-PI*360/180}" soft_upper_limit="${PI*360/180}"/>
+      <limit acceleration="15" effort="500.0" lower="${-PI*360/180}" upper="${PI*360/180}" velocity="${180/180*PI}"/>
+      <parent link="${arm_id}_link5"/>
+      <child link="${arm_id}_link6"/>
+      <dynamics D="1" K="7000" mu_coulomb="0" mu_viscous="16" damping="0.003" friction="0.01"/>
+    </joint>
+    <!-- joint6 -->
+    <joint name="${arm_id}_joint6" type="fixed">
+      <origin xyz="0.0 0.0 ${joint6_z}" rpy="0.0 0.0 0.0"/>
+      <parent link="${arm_id}_link6"/>
+      <child link="${arm_id}_link7"/>
+    </joint>
   </xacro:macro>
 </robot>

File: src/elephant/elerobot_description/xacro/property.xacro (robot description, xacro)
@@ -15,5 +15,9 @@
   <xacro:property name="link5_mass" value="1.417"/>
   <xacro:property name="link6_mass" value="0.3158"/>
-  <!-- link position -->
+  <xacro:property name="link7_mass" value="0.1"/>
+  <!-- link property -->
+  <xacro:property name="link7_r" value="0.05"/>
+  <xacro:property name="link7_h" value="0.08"/>
+  <!-- joint position -->
   <xacro:property name="joint0_z" value="0.107"/>
   <xacro:property name="joint1_y" value="0.05"/>
@@ -21,5 +25,14 @@
   <xacro:property name="joint3_x" value="0.238"/>
   <xacro:property name="joint3_z" value="0.063"/>
-  <xacro:property name="joint4_y" value="-0.097"/>
+  <xacro:property name="joint4_y" value="-0.095"/>
+  <xacro:property name="joint5_y" value="0.06"/>
+  <xacro:property name="joint6_z" value="${link7_h+0.032}"/>
+  <!-- inertia -->
+  <xacro:macro name="cylinder_inertia" params="m r h">
+    <inertia  ixx="${m*(3*r*r+h*h)/12}" ixy = "0" ixz = "0"
+      iyy="${m*(3*r*r+h*h)/12}" iyz = "0"
+      izz="${m*r*r/2}"
+    />
+  </xacro:macro>
   <!-- MACRO: transmission of the joint-->
   <![CDATA[

Commit message: add vaccum gripper group with 13 parts

File: src/elephant/elerobot_description/xacro/elerobot.xacro (robot description, xacro)
@@ -4,4 +4,5 @@
   <xacro:include filename="$(find elerobot_description)/xacro/color.xacro"/>
   <xacro:include filename="$(find elerobot_description)/xacro/property.xacro"/>
+  <xacro:include filename="$(find elerobot_description)/xacro/vacuum_group.xacro"/>
   <!-- elephant panda robot p3 type description-->
   <xacro:macro name="elerobot" params="arm_id:='elerobot' with_camera:='false'">
@@ -269,4 +270,18 @@
       <child link="${arm_id}_link7"/>
     </joint>
+    <!-- vacuum gripper -->
+    <xacro:vacuum_group parent_link="${arm_id}_link7" index="1" vacuum_x="0"                    vacuum_y="0"                   vacuum_z="${vacuum_length/2}"/>
+    <xacro:vacuum_group parent_link="${arm_id}_link7" index="2" vacuum_x="${vacuum_radius*3}"   vacuum_y="0"                   vacuum_z="${vacuum_length/2}"/>
+    <xacro:vacuum_group parent_link="${arm_id}_link7" index="3" vacuum_x="${-vacuum_radius*3}"  vacuum_y="0"                   vacuum_z="${vacuum_length/2}"/>
+    <xacro:vacuum_group parent_link="${arm_id}_link7" index="4" vacuum_x="0"                    vacuum_y="${vacuum_radius*3}"  vacuum_z="${vacuum_length/2}"/>
+    <xacro:vacuum_group parent_link="${arm_id}_link7" index="5" vacuum_x="0"                    vacuum_y="${-vacuum_radius*3}" vacuum_z="${vacuum_length/2}"/>
+    <xacro:vacuum_group parent_link="${arm_id}_link7" index="6" vacuum_x="${vacuum_radius*6}"   vacuum_y="0"                   vacuum_z="${vacuum_length/2}"/>
+    <xacro:vacuum_group parent_link="${arm_id}_link7" index="7" vacuum_x="${-vacuum_radius*6}"  vacuum_y="0"                   vacuum_z="${vacuum_length/2}"/>
+    <xacro:vacuum_group parent_link="${arm_id}_link7" index="8" vacuum_x="0"                    vacuum_y="${vacuum_radius*6}"  vacuum_z="${vacuum_length/2}"/>
+    <xacro:vacuum_group parent_link="${arm_id}_link7" index="9" vacuum_x="0"                    vacuum_y="${-vacuum_radius*6}" vacuum_z="${vacuum_length/2}"/>
+    <xacro:vacuum_group parent_link="${arm_id}_link7" index="10" vacuum_x="${vacuum_radius*4}"  vacuum_y="${vacuum_radius*4}"  vacuum_z="${vacuum_length/2}"/>
+    <xacro:vacuum_group parent_link="${arm_id}_link7" index="11" vacuum_x="${-vacuum_radius*4}" vacuum_y="${-vacuum_radius*4}" vacuum_z="${vacuum_length/2}"/>
+    <xacro:vacuum_group parent_link="${arm_id}_link7" index="12" vacuum_x="${-vacuum_radius*4}" vacuum_y="${vacuum_radius*4}"  vacuum_z="${vacuum_length/2}"/>
+    <xacro:vacuum_group parent_link="${arm_id}_link7" index="13" vacuum_x="${vacuum_radius*4}"  vacuum_y="${-vacuum_radius*4}" vacuum_z="${vacuum_length/2}"/>
   </xacro:macro>
 </robot>

File: src/elephant/elerobot_description/xacro/property.xacro (robot description, xacro)
@@ -19,4 +19,7 @@
   <xacro:property name="link7_r" value="0.05"/>
   <xacro:property name="link7_h" value="0.08"/>
+  <!-- vaccum property -->
+  <xacro:property name="vacuum_radius" value="0.005"/>
+  <xacro:property name="vacuum_length" value="0.005"/>
   <!-- joint position -->
   <xacro:property name="joint0_z" value="0.107"/>

File: src/elephant/elerobot_description/xacro/vacuum_group.xacro (robot description, xacro)
@@ -1,5 +1,4 @@
 <?xml version="1.0"?>
 <robot xmlns:xacro="http://www.ros.org/wiki/xacro" name="rokae_arm">
-  <xacro:include filename="$(find rokae_description)/xacro/macros.xacro"/>
   <xacro:macro name="vacuum_group" params="parent_link index vacuum_x vacuum_y vacuum_z">
     <xacro:property name="vacuum_gripper" value="vacuum_gripper_${index}"/>

Commit message: create ikfast solver (with plugin); create elerobot_moveit_config; add realsense camera for robot

File: src/elephant/elerobot_description/xacro/elerobot.xacro (robot description, xacro)
@@ -7,4 +7,11 @@
   <!-- elephant panda robot p3 type description-->
   <xacro:macro name="elerobot" params="arm_id:='elerobot' with_camera:='false'">
+    <!-- di435  frame definition can be found at https://github.com/IntelRealSense/librealsense/blob/master/doc/d435i.md -->
+    <xacro:if value="${with_camera}">
+      <xacro:include filename="$(find realsense_gazebo_description)/urdf/_d435i.urdf.xacro"/>
+      <xacro:sensor_d435i  parent="${arm_id}_link7" name="D435i_camera" topics_ns="D435i_camera" enable_pointCloud="true" align_depth="false">
+        <origin xyz="0.0 0.0 0.0" rpy="0.0 ${-PI/2} ${PI/2}"/>
+      </xacro:sensor_d435i>
+    </xacro:if>
     <!-- LINK DESCRIPTION -->
     <!-- Gazebo requires a joint to a link called "world" for statically mounted robots -->
@@ -49,5 +56,5 @@
       </visual>
       <collision>
-        <origin xyz="-0.051 -0.051 -0.07" rpy="0.0 0.0 0.0"/>
+        <origin xyz="-0.0528 -0.0528 -0.07" rpy="0.0 0.0 0.0"/>
         <geometry>
           <mesh filename="${mesh_file_path}${mesh_prefix}1${mesh_suffix}" scale="0.001 0.001 0.001"/>
@@ -192,5 +199,5 @@
       </visual>
       <collision>
-        <origin xyz="0.0 0.0 0.0" rpy="0.0 0.0 0.0"/>
+        <origin xyz="0.0 0.0 ${-link7_h/2}" rpy="0.0 0.0 0.0"/>
         <geometry>
           <cylinder radius="${link7_r}" length="${link7_h}"/>
@@ -204,9 +211,10 @@
     </link>
     <!-- JOINT DESCRIPTION -->
-    <!-- joint0 -->
+    <!-- joint0 Locked -->
     <joint name="${arm_id}_joint0" type="revolute">
       <axis xyz="0 0 1"/>
       <origin xyz="0.0 0.0 ${joint0_z}" rpy="0.0 0.0 0.0"/>
-      <safety_controller k_position="50.0" k_velocity="20.0" soft_lower_limit="${-PI*360/180}" soft_upper_limit="${PI*360/180}"/>
+      <safety_controller k_position="50.0" k_velocity="20.0" soft_lower_limit="${-PI*0.01/180}" soft_upper_limit="${PI*0.01/180}"/>
+      <!-- <safety_controller k_position="50.0" k_velocity="20.0" soft_lower_limit="${-PI*360/180}" soft_upper_limit="${PI*360/180}"/> -->
       <limit acceleration="15" effort="500.0" lower="${-PI*360/180}" upper="${PI*360/180}" velocity="${180/180*PI}"/>
       <parent link="${arm_id}_link0"/>
@@ -239,5 +247,5 @@
       <origin xyz="${joint3_x} 0.0 ${joint3_z}" rpy="0.0 0.0 ${PI/2}"/>
       <safety_controller k_position="50.0" k_velocity="20.0" soft_lower_limit="${-PI*360/180}" soft_upper_limit="${PI*360/180}"/>
-      <limit acceleration="15" effort="500.0" lower="${-PI*360/180}" upper="${PI*360/180}" velocity="${180/180*PI}"/>
+      <limit acceleration="15" effort="500.0" lower="${-PI*360/180}" upper="${PI*360/180}" velocity="${208/180*PI}"/>
       <parent link="${arm_id}_link3"/>
       <child link="${arm_id}_link4"/>
@@ -248,16 +256,17 @@
       <axis xyz="0 0 1"/>
       <origin xyz="0.0 ${joint4_y} 0.0" rpy="0.0 ${-PI/2} ${PI/2}"/>
-      <safety_controller k_position="50.0" k_velocity="20.0" soft_lower_limit="${-PI*360/180}" soft_upper_limit="${PI*360/180}"/>
-      <limit acceleration="15" effort="500.0" lower="${-PI*360/180}" upper="${PI*360/180}" velocity="${180/180*PI}"/>
+      <safety_controller k_position="50.0" k_velocity="20.0" soft_lower_limit="${-PI*0.01/180}" soft_upper_limit="${PI*0.01/180}"/>
+      <!-- <safety_controller k_position="50.0" k_velocity="20.0" soft_lower_limit="${-PI*360/180}" soft_upper_limit="${PI*360/180}"/> -->
+      <limit acceleration="15" effort="500.0" lower="${-PI*360/180}" upper="${PI*360/180}" velocity="${208/180*PI}"/>
       <parent link="${arm_id}_link4"/>
       <child link="${arm_id}_link5"/>
       <dynamics D="1" K="7000" mu_coulomb="0" mu_viscous="16" damping="0.003" friction="0.01"/>
     </joint>
-    <!-- joint5 -->
+    <!-- joint5 Locked -->
     <joint name="${arm_id}_joint5" type="revolute">
       <axis xyz="0 0 1"/>
       <origin xyz="0.0 ${joint5_y} 0.0" rpy="${-PI/2} 0.0 0.0"/>
       <safety_controller k_position="50.0" k_velocity="20.0" soft_lower_limit="${-PI*360/180}" soft_upper_limit="${PI*360/180}"/>
-      <limit acceleration="15" effort="500.0" lower="${-PI*360/180}" upper="${PI*360/180}" velocity="${180/180*PI}"/>
+      <limit acceleration="15" effort="500.0" lower="${-PI*360/180}" upper="${PI*360/180}" velocity="${208/180*PI}"/>
       <parent link="${arm_id}_link5"/>
       <child link="${arm_id}_link6"/>
