Commit message: load octomap

File: src/elephant/elerobot_description/xacro/elerobot.urdf.xacro (robot description, xacro)
@@ -4,5 +4,6 @@
   <xacro:arg name="gazebo" default="true" />
   <!-- Intel RealSense i435 -->
-  <xacro:arg name="with_camera" default="true" />
+  <!-- <xacro:arg name="with_camera" default="true" /> -->
+  <xacro:arg name="with_camera" default="false" />
   <!-- Robot name -->
   <xacro:property name="arm_id" value="elerobot" />

File: src/elephant/elerobot_description/xacro/elerobot.xacro (robot description, xacro)
@@ -196,5 +196,5 @@
           <cylinder radius="${link7_r}" length="${link7_h}"/>
         </geometry>
-        <material name="red"/>
+        <material name="orange"/>
       </visual>
       <collision>
