Commit message: update robot description to solve the end effector depature the gird; In rokae_arm_eef_state.cpp updates the data type for return value, otherwise the value will have a wired bias

File: src/elephant/elerobot_description/xacro/elerobot.urdf (robot description, URDF)
Before this commit: robot elerobot, 22 links, 21 joints
Links:
- link elerobot_link7: geometry collision cylinder length=0.04 radius=0.05; visual cylinder length=0.04 radius=0.05
Joints:
- joint elerobot_joint0: origin xyz=0.0 0.0 0.107 rpy=0.0 0.0 0.0 -> xyz=0.0 0.0 0.11 rpy=0.0 0.0 0.0
- joint elerobot_joint3: origin xyz=0.238 0.0 0.063 rpy=0.0 0.0 1.57079632675 -> xyz=0.24 0.0 0.06 rpy=0.0 0.0 1.57079632675
- joint elerobot_joint6: origin xyz=0.0 0.0 0.112 rpy=0.0 0.0 0.0 -> xyz=0.0 0.0 0.07 rpy=0.0 0.0 0.0

File: src/elephant/elerobot_description/xacro/elerobot.xacro (robot description, xacro)
@@ -73,5 +73,5 @@
     <link name="${arm_id}_link2">
       <visual>
-        <origin xyz="-0.054 -0.053 0.154" rpy="${-PI/2} 0.0 0.0"/>
+        <origin xyz="-0.054 -0.053 0.155" rpy="${-PI/2} 0.0 0.0"/>
         <geometry>
           <mesh filename="${mesh_file_path}${mesh_prefix}2${mesh_suffix}" scale="0.001 0.001 0.001"/>
@@ -80,5 +80,5 @@
       </visual>
       <collision>
-        <origin xyz="-0.054 -0.053 0.154" rpy="${-PI/2} 0.0 0.0"/>
+        <origin xyz="-0.054 -0.053 0.155" rpy="${-PI/2} 0.0 0.0"/>
         <geometry>
           <mesh filename="${mesh_file_path}${mesh_prefix}2${mesh_suffix}" scale="0.001 0.001 0.001"/>
@@ -97,5 +97,5 @@
     <link name="${arm_id}_link3">
       <visual>
-        <origin xyz="0.2815 0.078 0.024" rpy="${-PI/2} 0.0 ${PI}"/>
+        <origin xyz="0.2815 0.078 0.022" rpy="${-PI/2} 0.0 ${PI}"/>
         <geometry>
           <mesh filename="${mesh_file_path}${mesh_prefix}3${mesh_suffix}" scale="0.001 0.001 0.001"/>
@@ -104,5 +104,5 @@
       </visual>
       <collision>
-        <origin xyz="0.2815 0.078 0.024" rpy="${-PI/2} 0.0 ${PI}"/>
+        <origin xyz="0.2815 0.078 0.022" rpy="${-PI/2} 0.0 ${PI}"/>
         <geometry>
           <mesh filename="${mesh_file_path}${mesh_prefix}3${mesh_suffix}" scale="0.001 0.001 0.001"/>
@@ -121,5 +121,5 @@
     <link name="${arm_id}_link4">
       <visual>
-        <origin xyz="-0.0772 -0.0596 0.044" rpy="${-PI/2} 0.0 0.0"/>
+        <origin xyz="-0.0772 -0.055 0.046" rpy="${-PI/2} 0.0 0.0"/>
         <geometry>
           <mesh filename="${mesh_file_path}${mesh_prefix}4${mesh_suffix}" scale="0.001 0.001 0.001"/>
@@ -128,5 +128,5 @@
       </visual>
       <collision>
-        <origin xyz="-0.0772 -0.0596 0.044" rpy="${-PI/2} 0.0 0.0"/>
+        <origin xyz="-0.0772 -0.055 0.046" rpy="${-PI/2} 0.0 0.0"/>
         <geometry>
           <mesh filename="${mesh_file_path}${mesh_prefix}4${mesh_suffix}" scale="0.001 0.001 0.001"/>
@@ -215,6 +215,6 @@
       <axis xyz="0 0 1"/>
       <origin xyz="0.0 0.0 ${joint0_z}" rpy="0.0 0.0 0.0"/>
-      <safety_controller k_position="50.0" k_velocity="20.0" soft_lower_limit="${-PI*0.01/180}" soft_upper_limit="${PI*0.01/180}"/>
-      <!-- <safety_controller k_position="50.0" k_velocity="20.0" soft_lower_limit="${-PI*360/180}" soft_upper_limit="${PI*360/180}"/> -->
+      <!-- <safety_controller k_position="50.0" k_velocity="20.0" soft_lower_limit="${-PI*0.001/180}" soft_upper_limit="${PI*0.001/180}"/> -->
+      <safety_controller k_position="50.0" k_velocity="20.0" soft_lower_limit="${-PI*360/180}" soft_upper_limit="${PI*360/180}"/>
       <limit acceleration="15" effort="500.0" lower="${-PI*360/180}" upper="${PI*360/180}" velocity="${180/180*PI}"/>
       <parent link="${arm_id}_link0"/>
@@ -256,6 +256,6 @@
       <axis xyz="0 0 1"/>
       <origin xyz="0.0 ${joint4_y} 0.0" rpy="0.0 ${-PI/2} ${PI/2}"/>
-      <safety_controller k_position="50.0" k_velocity="20.0" soft_lower_limit="${-PI*0.01/180}" soft_upper_limit="${PI*0.01/180}"/>
-      <!-- <safety_controller k_position="50.0" k_velocity="20.0" soft_lower_limit="${-PI*360/180}" soft_upper_limit="${PI*360/180}"/> -->
+      <!-- <safety_controller k_position="50.0" k_velocity="20.0" soft_lower_limit="${-PI*0.001/180}" soft_upper_limit="${PI*0.001/180}"/> -->
+      <safety_controller k_position="50.0" k_velocity="20.0" soft_lower_limit="${-PI*360/180}" soft_upper_limit="${PI*360/180}"/>
       <limit acceleration="15" effort="500.0" lower="${-PI*360/180}" upper="${PI*360/180}" velocity="${208/180*PI}"/>
       <parent link="${arm_id}_link4"/>

File: src/elephant/elerobot_description/xacro/property.xacro (robot description, xacro)
@@ -18,17 +18,17 @@
   <!-- link property -->
   <xacro:property name="link7_r" value="0.05"/>
-  <xacro:property name="link7_h" value="0.08"/>
+  <xacro:property name="link7_h" value="0.04"/>
   <!-- vaccum property -->
   <xacro:property name="vacuum_radius" value="0.005"/>
   <xacro:property name="vacuum_length" value="0.005"/>
   <!-- joint position -->
-  <xacro:property name="joint0_z" value="0.107"/>
+  <xacro:property name="joint0_z" value="0.11"/>
   <xacro:property name="joint1_y" value="0.05"/>
   <xacro:property name="joint2_x" value="0.265"/>
-  <xacro:property name="joint3_x" value="0.238"/>
-  <xacro:property name="joint3_z" value="0.063"/>
+  <xacro:property name="joint3_x" value="0.24"/>
+  <xacro:property name="joint3_z" value="0.06"/>
   <xacro:property name="joint4_y" value="-0.095"/>
   <xacro:property name="joint5_y" value="0.06"/>
-  <xacro:property name="joint6_z" value="${link7_h+0.032}"/>
+  <xacro:property name="joint6_z" value="${link7_h+0.03}"/>
   <!-- inertia -->
   <xacro:macro name="cylinder_inertia" params="m r h">

Commit message: sovle the planning problem; re-understand the octomap voxel property especially the point3d position

File: src/elephant/elerobot_description/xacro/elerobot.urdf (robot description, URDF)
Before this commit: robot elerobot, 22 links, 21 joints
Joints:
- joint elerobot_joint0: origin xyz=0.0 0.0 0.11 rpy=0.0 0.0 0.0 -> xyz=0.0 0.0 0.115 rpy=0.0 0.0 0.0
- joint elerobot_joint1: origin xyz=0.0 0.05 0.0 rpy=0.0 -1.57079632675 -1.57079632675 -> xyz=0.0 0.055 0.0 rpy=0.0 -1.57079632675 -1.57079632675
- joint world_joint: origin xyz=0.0 0.0 0.0 rpy=0.0 0.0 0.0 -> xyz=0.005 0.0 0.0 rpy=0.0 0.0 0.0

File: src/elephant/elerobot_description/xacro/elerobot.xacro (robot description, xacro)
@@ -18,5 +18,5 @@
     <link name="world" />
     <joint name="world_joint" type="fixed">
-      <origin xyz="0.0 0.0 0.0" rpy="0.0 0.0 0.0"/>
+      <origin xyz="0.005 0.0 0.0" rpy="0.0 0.0 0.0"/>
       <parent link="world"/>
       <child link="${arm_id}_link0"/>
@@ -25,5 +25,5 @@
     <link name="${arm_id}_link0">
       <visual>
-        <origin xyz="-0.06 -0.06 0.05" rpy="${-PI/2} 0.0 0.0"/>
+        <origin xyz="-0.06 -0.06 0.053" rpy="${-PI/2} 0.0 0.0"/>
         <geometry>
           <mesh filename="${mesh_file_path}${mesh_prefix}0${mesh_suffix}" scale="0.001 0.001 0.001"/>
@@ -32,5 +32,5 @@
       </visual>
       <collision>
-        <origin xyz="-0.06 -0.06 0.05" rpy="${-PI/2} 0.0 0.0"/>
+        <origin xyz="-0.06 -0.06 0.053" rpy="${-PI/2} 0.0 0.0"/>
         <geometry>
           <mesh filename="${mesh_file_path}${mesh_prefix}0${mesh_suffix}" scale="0.001 0.001 0.001"/>
@@ -49,5 +49,5 @@
     <link name="${arm_id}_link1">
       <visual>
-        <origin xyz="-0.0528 -0.0528 -0.07" rpy="0.0 0.0 0.0"/>
+        <origin xyz="-0.0528 -0.0528 -0.072" rpy="0.0 0.0 0.0"/>
         <geometry>
           <mesh filename="${mesh_file_path}${mesh_prefix}1${mesh_suffix}" scale="0.001 0.001 0.001"/>
@@ -56,5 +56,5 @@
       </visual>
       <collision>
-        <origin xyz="-0.0528 -0.0528 -0.07" rpy="0.0 0.0 0.0"/>
+        <origin xyz="-0.0528 -0.0528 -0.072" rpy="0.0 0.0 0.0"/>
         <geometry>
           <mesh filename="${mesh_file_path}${mesh_prefix}1${mesh_suffix}" scale="0.001 0.001 0.001"/>
@@ -73,5 +73,5 @@
     <link name="${arm_id}_link2">
       <visual>
-        <origin xyz="-0.054 -0.053 0.155" rpy="${-PI/2} 0.0 0.0"/>
+        <origin xyz="-0.054 -0.053 0.15" rpy="${-PI/2} 0.0 0.0"/>
         <geometry>
           <mesh filename="${mesh_file_path}${mesh_prefix}2${mesh_suffix}" scale="0.001 0.001 0.001"/>
@@ -80,5 +80,5 @@
       </visual>
       <collision>
-        <origin xyz="-0.054 -0.053 0.155" rpy="${-PI/2} 0.0 0.0"/>
+        <origin xyz="-0.054 -0.053 0.15" rpy="${-PI/2} 0.0 0.0"/>
         <geometry>
           <mesh filename="${mesh_file_path}${mesh_prefix}2${mesh_suffix}" scale="0.001 0.001 0.001"/>
@@ -97,5 +97,5 @@
     <link name="${arm_id}_link3">
       <visual>
-        <origin xyz="0.2815 0.078 0.022" rpy="${-PI/2} 0.0 ${PI}"/>
+        <origin xyz="0.2815 0.078 0.017" rpy="${-PI/2} 0.0 ${PI}"/>
         <geometry>
           <mesh filename="${mesh_file_path}${mesh_prefix}3${mesh_suffix}" scale="0.001 0.001 0.001"/>
@@ -104,5 +104,5 @@
       </visual>
       <collision>
-        <origin xyz="0.2815 0.078 0.022" rpy="${-PI/2} 0.0 ${PI}"/>
+        <origin xyz="0.2815 0.078 0.017" rpy="${-PI/2} 0.0 ${PI}"/>
         <geometry>
           <mesh filename="${mesh_file_path}${mesh_prefix}3${mesh_suffix}" scale="0.001 0.001 0.001"/>
@@ -121,5 +121,5 @@
     <link name="${arm_id}_link4">
       <visual>
-        <origin xyz="-0.0772 -0.055 0.046" rpy="${-PI/2} 0.0 0.0"/>
+        <origin xyz="-0.0772 -0.055 0.043" rpy="${-PI/2} 0.0 0.0"/>
         <geometry>
           <mesh filename="${mesh_file_path}${mesh_prefix}4${mesh_suffix}" scale="0.001 0.001 0.001"/>
@@ -128,5 +128,5 @@
       </visual>
       <collision>
-        <origin xyz="-0.0772 -0.055 0.046" rpy="${-PI/2} 0.0 0.0"/>
+        <origin xyz="-0.0772 -0.055 0.043" rpy="${-PI/2} 0.0 0.0"/>
         <geometry>
           <mesh filename="${mesh_file_path}${mesh_prefix}4${mesh_suffix}" scale="0.001 0.001 0.001"/>
@@ -145,5 +145,5 @@
     <link name="${arm_id}_link5">
       <visual>
-        <origin xyz="0.0775 0.0605 0.046" rpy="${-PI/2} 0.0 ${PI}"/>
+        <origin xyz="0.0745 0.0605 0.046" rpy="${-PI/2} 0.0 ${PI}"/>
         <geometry>
           <mesh filename="${mesh_file_path}${mesh_prefix}5${mesh_suffix}" scale="0.001 0.001 0.001"/>
@@ -152,5 +152,5 @@
       </visual>
       <collision>
-        <origin xyz="0.0775 0.0605 0.046" rpy="${-PI/2} 0.0 ${PI}"/>
+        <origin xyz="0.0745 0.0605 0.046" rpy="${-PI/2} 0.0 ${PI}"/>
         <geometry>
           <mesh filename="${mesh_file_path}${mesh_prefix}5${mesh_suffix}" scale="0.001 0.001 0.001"/>

File: src/elephant/elerobot_description/xacro/property.xacro (robot description, xacro)
@@ -23,6 +23,6 @@
   <xacro:property name="vacuum_length" value="0.005"/>
   <!-- joint position -->
-  <xacro:property name="joint0_z" value="0.11"/>
-  <xacro:property name="joint1_y" value="0.05"/>
+  <xacro:property name="joint0_z" value="0.115"/>
+  <xacro:property name="joint1_y" value="0.055"/>
   <xacro:property name="joint2_x" value="0.265"/>
   <xacro:property name="joint3_x" value="0.24"/>

File: src/elephant/elerobot_description/xacro/vacuum_group.xacro (robot description, xacro)
@@ -38,4 +38,14 @@
       <dynamics damping="0.0" friction="10"/>
     </joint>
+    <![CDATA[
+    <joint name="${gripper_joint}" type="fixed">
+      <!-- <axis xyz="0 0 1" /> -->
+      <parent link="${parent_link}" />
+      <child link="${vacuum_gripper}" />
+      <origin rpy="0 0 0" xyz="${vacuum_x} ${vacuum_y} ${vacuum_z}" />
+      <!-- <limit effort="50" velocity="50" lower="0" upper="0" /> -->
+      <!-- <dynamics damping="0.0" friction="10"/> -->
+    </joint>
+    ]]>
     <gazebo>
       <plugin name="gazebo_ros_vacuum_gripper_${index}" filename="libgazebo_ros_vacuum_gripper.so">
